Commit message: models

File: Simulation/robot_arm/urdf/arm.xacro (robot description, xacro)
@@ -1,3 +1,2 @@
-<!-- arm2.xacro:- has inertia, collision properties for links for simulation in gazebo -->
 <?xml version="1.0" ?>
 <robot name="arm" xmlns:xacro="http://www.ros.org/wiki/xacro">
@@ -19,7 +18,7 @@
     <link name="base">
     <inertial>
-	    <mass value="1"/>
-	    <origin rpy="0 0 0" xyz="0 0 0"	/> 	<!--same as origin of link-->
-	    <inertia ixx="" ixy="0" ixz="0" iyy="" iyz="0" izz="" />
+	    <mass value=""/>
+	    <origin rpy="0 0 0" xyz="0 0 0"	/> 	<!--same as origin of link-->
+	    <inertia ixx="" ixy="" ixz="" iyy="" iyz="" izz="" />
     </inertial>
     <collision>
@@ -47,7 +46,7 @@
     <link name="servo1">
     <inertial>
-	    <mass value="0.250"/>
+	    <mass value=""/>
 	    <origin rpy="0 0 0" xyz="0 0 0.1"	/> 	<!--same as origin of link-->
-	    <inertia ixx="" ixy="0" ixz="0" iyy="" iyz="0" izz="" />
+	    <inertia ixx="" ixy="" ixz="" iyy="" iyz="" izz="" />
     </inertial>
         <collision>
@@ -75,7 +74,7 @@
     <link name="shaft1">
     <inertial>
-	    <mass value="0.050"/>
-	    <origin rpy="0 0 0" xyz="0 0 0"	/> 	<!--same as origin of link-->
-	    <inertia ixx="" ixy="0" ixz="0" iyy="" iyz="0" izz=""/>
+	    <mass value=""/>
+	    <origin rpy="0 0 0" xyz="0 0 0"	/> 	<!--same as origin of link-->
+	    <inertia ixx="" ixy="" ixz="" iyy="" iyz="" izz="" />
     </inertial>
     <collision>
@@ -102,7 +101,7 @@
     <link name="link1">
     <inertial>
-	    <mass value="0.100"/>
-	    <origin rpy="0 0 0" xyz="0 0 0"	/> 	<!--same as origin of link-->
-	    <inertia ixx="" ixy="0" ixz="0" iyy="" iyz="0" izz=""/>
+	    <mass value=""/>
+	    <origin rpy="0 0 0" xyz="0 0 0"	/> 	<!--same as origin of link-->
+	    <inertia ixx="" ixy="" ixz="" iyy="" iyz="" izz="" />
     </inertial>
     <collision>
@@ -129,7 +128,7 @@
     <link name="servo2">
     <inertial>
-	    <mass value="0.250"/>
-	    <origin rpy="0 0 0" xyz="0 0 0"	/> 	<!--same as origin of link-->
-	    <inertia ixx="" ixy="0" ixz="0" iyy="" iyz="0" izz=""/>
+	    <mass value=""/>
+	    <origin rpy="0 0 0" xyz="0 0 0"	/> 	<!--same as origin of link-->
+	    <inertia ixx="" ixy="" ixz="" iyy="" iyz="" izz="" />
     </inertial>
     <collision>
@@ -157,7 +156,7 @@
     <link name="shaft2">
     <inertial>
-	    <mass value="0.050"/>
-	    <origin rpy="0 0 0" xyz="0 0 0"	/> 	<!--same as origin of link-->
-	    <inertia ixx="" ixy="0" ixz="0" iyy="" iyz="0" izz="" />
+	    <mass value=""/>
+	    <origin rpy="0 0 0" xyz="0 0 0"	/> 	<!--same as origin of link-->
+	    <inertia ixx="" ixy="" ixz="" iyy="" iyz="" izz="" />
     </inertial>
     <collision>
@@ -184,5 +183,5 @@
     <link name="link2">
     <inertial>
-	    <mass value="0.100"/>
+	    <mass value=""/>
 	    <origin rpy="0 0 0" xyz="0 0 0"	/> 	<!--same as origin of link-->
 	    <inertia ixx="" ixy="" ixz="" iyy="" iyz="" izz="" />
@@ -211,5 +210,5 @@
     <link name="servo3">
     <inertial>
-	    <mass value="0.250"/>
+	    <mass value=""/>
 	    <origin rpy="0 0 0" xyz="0 0 0"	/> 	<!--same as origin of link-->
 	    <inertia ixx="" ixy="" ixz="" iyy="" iyz="" izz="" />
@@ -239,5 +238,5 @@
     <link name="shaft3">
     <inertial>
-	    <mass value="0.050"/>
+	    <mass value=""/>
 	    <origin rpy="0 0 0" xyz="0 0 0"	/> 	<!--same as origin of link-->
 	    <inertia ixx="" ixy="" ixz="" iyy="" iyz="" izz="" />
@@ -266,5 +265,5 @@
     <link name="link3">
     <inertial>
-	    <mass value="0.100"/>
+	    <mass value=""/>
 	    <origin rpy="0 0 0" xyz="0 0 0"	/> 	<!--same as origin of link-->
 	    <inertia ixx="" ixy="" ixz="" iyy="" iyz="" izz="" />
@@ -293,5 +292,5 @@
     <link name="motor1">
     <inertial>
-	    <mass value="0.200"/>
+	    <mass value=""/>
 	    <origin rpy="0 0 0" xyz="0 0 0"	/> 	<!--same as origin of link-->
 	    <inertia ixx="" ixy="" ixz="" iyy="" iyz="" izz="" />
@@ -321,5 +320,5 @@
     <link name="shaft4">
     <inertial>
-	    <mass value="0.050"/>
+	    <mass value=""/>
 	    <origin rpy="0 0 0" xyz="0 0 0"	/> 	<!--same as origin of link-->
 	    <inertia ixx="" ixy="" ixz="" iyy="" iyz="" izz="" />
@@ -348,5 +347,5 @@
     <link name="brush">
     <inertial>
-	    <mass value="0.100"/>
+	    <mass value=""/>
 	    <origin rpy="0 0 0" xyz="0 0 0"	/> 	<!--same as origin of link-->
 	    <inertia ixx="" ixy="" ixz="" iyy="" iyz="" izz="" />
@@ -376,5 +375,5 @@
     <link name="base2">
     <inertial>
-	    <mass value="0.600"/>
+	    <mass value=""/>
 	    <origin rpy="0 0 0" xyz="0 0 0"	/> 	<!--same as origin of link-->
 	    <inertia ixx="" ixy="" ixz="" iyy="" iyz="" izz="" />
@@ -404,5 +403,5 @@
     <link name="servo2.1">
     <inertial>
-	    <mass value="0.250"/>
+	    <mass value=""/>
 	    <origin rpy="0 0 0" xyz="0 0 0"	/> 	<!--same as origin of link-->
 	    <inertia ixx="" ixy="" ixz="" iyy="" iyz="" izz="" />
@@ -432,5 +431,5 @@
     <link name="shaft2.1">
     <inertial>
-	    <mass value="0.050"/>
+	    <mass value=""/>
 	    <origin rpy="0 0 0" xyz="0 0 0"	/> 	<!--same as origin of link-->
 	    <inertia ixx="" ixy="" ixz="" iyy="" iyz="" izz="" />
@@ -459,5 +458,5 @@
     <link name="link2.1">
     <inertial>
-	    <mass value="0.100"/>
+	    <mass value=""/>
 	    <origin rpy="0 0 0" xyz="0 0 0"	/> 	<!--same as origin of link-->
 	    <inertia ixx="" ixy="" ixz="" iyy="" iyz="" izz="" />
@@ -486,5 +485,5 @@
     <link name="servo2.2">
     <inertial>
-	    <mass value="0.250"/>
+	    <mass value=""/>
 	    <origin rpy="0 0 0" xyz="0 0 0"	/> 	<!--same as origin of link-->
 	    <inertia ixx="" ixy="" ixz="" iyy="" iyz="" izz="" />
@@ -514,5 +513,5 @@
     <link name="shaft2.2">
     <inertial>
-	    <mass value="0.050"/>
+	    <mass value=""/>
 	    <origin rpy="0 0 0" xyz="0 0 0"	/> 	<!--same as origin of link-->
 	    <inertia ixx="" ixy="" ixz="" iyy="" iyz="" izz="" />
@@ -542,5 +541,5 @@
     <link name="left_gripper">
     <inertial>
-	    <mass value="0.075"/>
+	    <mass value=""/>
 	    <origin rpy="0 0 0" xyz="0 0 0"	/> 	<!--same as origin of link-->
 	    <inertia ixx="" ixy="" ixz="" iyy="" iyz="" izz="" />
@@ -565,5 +564,5 @@
   <link name="left_tip">
   <inertial>
-	    <mass value="0.020"/>
+	    <mass value=""/>
 	    <origin rpy="0 0 0" xyz="0 0 0"	/> 	<!--same as origin of link-->
 	    <inertia ixx="" ixy="" ixz="" iyy="" iyz="" izz="" />
@@ -591,5 +590,5 @@
   <link name="right_gripper">
   <inertial>
-	    <mass value="0.075"/>
+	    <mass value=""/>
 	    <origin rpy="0 0 0" xyz="0 0 0"	/> 	<!--same as origin of link-->
 	    <inertia ixx="" ixy="" ixz="" iyy="" iyz="" izz="" />
@@ -614,5 +613,5 @@
   <link name="right_tip">
   <inertial>
-	    <mass value="0.020"/>
+	    <mass value=""/>
 	    <origin rpy="0 0 0" xyz="0 0 0"	/> 	<!--same as origin of link-->
 	    <inertia ixx="" ixy="" ixz="" iyy="" iyz="" izz="" />
@@ -631,8 +630,3 @@
     </visual>
   </link>
-  <!-- gazebo plugin -->
-   <gazebo>
-    <plugin name="gazebo_ros_control" filename="libgazebo_ros_control.so">
-    </plugin>
-   </gazebo>
 </robot>
